Commit message: type: feat 1.update the museum model. 2.add poster model. 3.move meshes/ to model/meshes

File: robot_sim_demo/urdf/sick_tim.urdf.xacro (robot description, xacro)
@@ -8,5 +8,5 @@
       length="0.06" width="0.06" height="0.079" mass="0.150" z_offset="0.05595"
       min_range="0.05" max_range="4.0"
-      mesh="package://robot_sim_demo/meshes/sick_tim310.stl" />
+      mesh="package://robot_sim_demo/models/meshes/sick_tim310.stl" />
   </xacro:macro>
   <xacro:macro name="sick_tim551" params="name ros_topic">
@@ -14,5 +14,5 @@
       length="0.06" width="0.06" height="0.086" mass="0.250" z_offset="0.06296"
       min_range="0.05" max_range="10.0"
-      mesh="package://robot_sim_demo/meshes/sick_tim551.stl" />
+      mesh="package://robot_sim_demo/models/meshes/sick_tim551.stl" />
   </xacro:macro>
   <xacro:macro name="sick_tim571" params="name ros_topic">
@@ -20,5 +20,5 @@
       length="0.06" width="0.06" height="0.086" mass="0.250" z_offset="0.02"
       min_range="0.05" max_range="25.0"
-      mesh="package://robot_sim_demo/meshes/sick_tim571.stl" />
+      mesh="package://robot_sim_demo/models/meshes/sick_tim571.stl" />
   </xacro:macro>
   <xacro:macro name="sick_tim" params="name ros_topic length width height mass z_offset min_range max_range mesh">

File: robot_sim_demo/urdf/xbot2.urdf.xacro (robot description, xacro)
@@ -21,5 +21,5 @@
       <origin xyz="0 0 0" rpy="0 0 0" />
       <geometry>
-        <mesh filename="package://robot_sim_demo/meshes/base_link.dae" />
+        <mesh filename="package://robot_sim_demo/models/meshes/base_link.dae" />
       </geometry>
     </visual>
@@ -78,5 +78,5 @@
       <origin xyz="0 0 0" rpy="0 0 -1.570796"/>
       <geometry>
-        <mesh filename="package://robot_sim_demo/meshes/wheel.dae" />
+        <mesh filename="package://robot_sim_demo/models/meshes/wheel.dae" />
       </geometry>
     </visual>
@@ -105,5 +105,5 @@
       <origin xyz="0 0 0" rpy="0 0 1.570796"/>
       <geometry>
-        <mesh filename="package://robot_sim_demo/meshes/wheel.dae" />
+        <mesh filename="package://robot_sim_demo/models/meshes/wheel.dae" />
       </geometry>
     </visual>
@@ -131,5 +131,5 @@
       <origin xyz="0 0 0" rpy="0 0 1.570796" />
       <geometry>
-        <mesh filename="package://robot_sim_demo/meshes/yaw_platform.stl" />
+        <mesh filename="package://robot_sim_demo/models/meshes/yaw_platform.stl" />
       </geometry>
       <material name="grey"/>
@@ -159,5 +159,5 @@
       <origin xyz="0 0 0" rpy="0 0 0" />
       <geometry>
-        <mesh filename="package://robot_sim_demo/meshes/pitch_platform.stl" />
+        <mesh filename="package://robot_sim_demo/models/meshes/pitch_platform.stl" />
       </geometry>
       <material name="grey"/>
@@ -189,5 +189,5 @@
       <origin xyz="0 0 0" rpy="0 0 0"/>
       <geometry>
-        <mesh filename="package://robot_sim_demo/meshes/xtion_pro_camera.dae" />
+        <mesh filename="package://robot_sim_demo/models/meshes/xtion_pro_camera.dae" />
       </geometry>
       <material name="gray"/>
