Commit message: fix a bug that  cannot be resolved properly in Indigo

File: robot_sim_demo/urdf/xbot2.urdf.xacro (robot description, xacro)
@@ -210,5 +210,5 @@
     <!-- these values have to be these values otherwise the gazebo camera image
         won't be aligned properly with the frame it is supposedly originating from -->
-    <origin xyz="0 0 0" rpy="${-pi/2} 0 ${-pi/2}"/>
+    <origin xyz="0 0 0" rpy="-1.5708 0 -1.5708"/>
     <parent link="camera_link"/>
     <child link="camera_link_optical"/>

Commit message: fix:modify (0,0,0) collision box to (0.1, 0.1, 0.1) to avoid gazebo crash

File: robot_sim_demo/urdf/xbot2.urdf.xacro (robot description, xacro)
@@ -138,5 +138,5 @@
       <origin xyz="0 0 0" rpy="0 0 1.570796" />
       <geometry>
-        <box size="0.0 0.0 0.0"/>
+        <box size="0.1 0.1 0.1"/>
       </geometry>
     </collision>
@@ -166,5 +166,5 @@
       <origin xyz="0 0 0" rpy="0 0 0" />
       <geometry>
-        <box size="0.0 0.0 0.0"/>
+        <box size="0.1 0.1 0.1"/>
       </geometry>
     </collision>
@@ -183,5 +183,5 @@
       <origin xyz="0 0 0" rpy="0 0 0"/>
       <geometry>
-        <box size="0.0 0.0 0.0"/>
+        <box size="0.1 0.1 0.1"/>
       </geometry>
     </collision>

Commit message: fix the the bug that laserscan on the obstacle model

File: robot_sim_demo/urdf/xbot2.urdf.xacro (robot description, xacro)
@@ -45,5 +45,5 @@
       <origin xyz="0.03 0 0.25" rpy="0 0 0" />
       <geometry>
-        <cylinder length="0.08" radius="0.15"/>
+        <cylinder length="0.08" radius="0.045"/>
       </geometry>
     </collision>

Commit message: update keyboard_teleop

File: robot_sim_demo/urdf/xbot2.urdf.xacro (robot description, xacro)
@@ -92,5 +92,5 @@
     <parent link="base_link"/>
     <child link="left_wheel"/>
-    <limit effort="100000" velocity="1000"/>
+    <limit effort="5.2" velocity="2.0"/>
     <joint_properties damping="0.0" friction="0.0"/>
   </joint>
@@ -119,5 +119,5 @@
     <parent link="base_link"/>
     <child link="right_wheel"/>
-    <limit effort="100000" velocity="1000"/>
+    <limit effort="5.2" velocity="2.0"/>
     <joint_properties damping="0.0" friction="0.0"/>
   </joint>

Commit message: add imu to robot

File: robot_sim_demo/urdf/xbot2.urdf.xacro (robot description, xacro)
@@ -68,4 +68,11 @@
     <origin rpy="0 3.1416 3.1416" xyz=".148 0 .253"/>
   </joint>
+  <link name="imu_link"/>
+  <joint name="base_to_imu" type="fixed">
+    <axis rpy="0 0 0" xyz="0 0 0"/>
+    <parent link="base_link"/>
+    <child link="imu_link"/>
+    <origin rpy="0 0 0" xyz="0 0 .2"/>
+  </joint>
   <link name="left_wheel">
     <collision name="collision">
