Commit message: type: fix replace simple_robot demo to robot_sim_demo, using xbot2 model

File: robot_sim_demo/urdf/robot.xacro (robot description, xacro)
@@ -5,10 +5,10 @@
   xmlns:xacro="http://ros.org/wiki/xacro"
   name="sick_tim">
-  <xacro:include filename="$(find robot_sim_demo)/urdf/sick_tim.urdf.xacro" />
+  <xacro:include filename="$(find xbot2_description)/urdf/sick_tim.urdf.xacro" />
   <xacro:sick_tim571 name="laser" ros_topic="scan"   />
-  <xacro:include filename="$(find robot_sim_demo)/urdf/materials.xacro" />
-  <xacro:include filename="$(find robot_sim_demo)/urdf/xbot2.urdf.xacro" />
-  <xacro:include filename="$(find robot_sim_demo)/urdf/xbot2.gazebo" />
+  <xacro:include filename="$(find xbot2_description)/urdf/materials.xacro" />
+  <xacro:include filename="$(find xbot2_description)/urdf/xbot2.urdf.xacro" />
+  <xacro:include filename="$(find xbot2_description)/urdf/xbot2.gazebo" />
   <xacro:xbot2_base/>
-  <!--xacro:include filename="$(find robot_sim_demo)/urdf/sick_tim.gazebo.xacro" /-->
+  <!--xacro:include filename="$(find xbot2_description)/urdf/sick_tim.gazebo.xacro" /-->
 </robot>

File: robot_sim_demo/urdf/sick_tim.urdf.xacro (robot description, xacro)
@@ -8,5 +8,5 @@
       length="0.06" width="0.06" height="0.079" mass="0.150" z_offset="0.05595"
       min_range="0.05" max_range="4.0"
-      mesh="package://robot_sim_demo/meshes/sick_tim310.stl" />
+      mesh="package://xbot2_description/meshes/sick_tim310.stl" />
   </xacro:macro>
   <xacro:macro name="sick_tim551" params="name ros_topic">
@@ -14,5 +14,5 @@
       length="0.06" width="0.06" height="0.086" mass="0.250" z_offset="0.06296"
       min_range="0.05" max_range="10.0"
-      mesh="package://robot_sim_demo/meshes/sick_tim551.stl" />
+      mesh="package://xbot2_description/meshes/sick_tim551.stl" />
   </xacro:macro>
   <xacro:macro name="sick_tim571" params="name ros_topic">
@@ -20,5 +20,5 @@
       length="0.06" width="0.06" height="0.086" mass="0.250" z_offset="0.02"
       min_range="0.05" max_range="25.0"
-      mesh="package://robot_sim_demo/meshes/sick_tim571.stl" />
+      mesh="package://xbot2_description/meshes/sick_tim571.stl" />
   </xacro:macro>
   <xacro:macro name="sick_tim" params="name ros_topic length width height mass z_offset min_range max_range mesh">

File: robot_sim_demo/urdf/xbot2.urdf.xacro (robot description, xacro)
@@ -14,18 +14,48 @@
   <link name="base_link">
     <inertial>
-      <origin  xyz="0 0 0.13" rpy="0 0 0" />
-      <mass value="25.0" />
-      <inertia ixx=".734" ixy="0" ixz="0" iyy=".734" iyz=".0" izz=".156" />
+      <origin  xyz="0.001 0 0.007" rpy="0 0 0" />
+      <mass value="30.0" />
+      <inertia ixx="1.734" ixy="0" ixz="0" iyy="1.734" iyz=".0" izz="1.0" />
     </inertial>
     <visual>
       <origin xyz="0 0 0" rpy="0 0 0" />
       <geometry>
-        <mesh filename="package://robot_sim_demo/meshes/base_link.dae" />
-      </geometry>
-    </visual>
-    <collision>
-      <origin xyz="0 0 0" rpy="0 0 0" />
-      <geometry>
-        <mesh filename="package://robot_sim_demo/meshes/base_link.dae" />
+        <mesh filename="package://xbot2_description/meshes/base_link.dae" />
+      </geometry>
+    </visual>
+    <collision name="front_omniwheel">
+      <origin xyz="0.18 0 0.02" rpy="0 0 0" />
+      <geometry>
+        <sphere radius="0.019"/>
+      </geometry>
+    </collision>
+    <collision name="back_omniwheel">
+      <origin xyz="-0.18 0 0.02" rpy="0 0 0" />
+      <geometry>
+        <sphere radius="0.019"/>
+      </geometry>
+    </collision>
+    <collision name="collision1">
+      <origin xyz="0.0 0 0.135" rpy="0 0 0" />
+      <geometry>
+        <cylinder length="0.15" radius="0.25"/>
+      </geometry>
+    </collision>
+    <collision name="collision2">
+      <origin xyz="0.03 0 0.25" rpy="0 0 0" />
+      <geometry>
+        <cylinder length="0.08" radius="0.15"/>
+      </geometry>
+    </collision>
+    <collision name="collision3">
+      <origin xyz="0 0 0.68" rpy="0 0 0" />
+      <geometry>
+        <cylinder length="0.8" radius="0.08"/>
+      </geometry>
+    </collision>
+    <collision name="collision4">
+      <origin xyz="0 0 1.135" rpy="0 0 0" />
+      <geometry>
+        <box size="0.04 0.17 0.09"/>
       </geometry>
     </collision>
@@ -40,17 +70,17 @@
   <link name="left_wheel">
     <collision name="collision">
-      <origin xyz="0 0 0" rpy="1.5708 0 0"/>
-      <geometry>
-        <cylinder radius="0.095" length="0.04"/>
+      <origin xyz="0 0 0" rpy="1.570796 0 0"/>
+      <geometry>
+        <cylinder radius="0.095" length="0.05"/>
       </geometry>
     </collision>
     <visual name="left_wheel_visual">
-      <origin xyz="0 0 0" rpy="0 0 -1.5708"/>
-      <geometry>
-        <mesh filename="package://robot_sim_demo/meshes/wheel.dae" />
-      </geometry>
-    </visual>
-    <inertial>
-      <origin xyz="0 0 0" rpy="0 0 -1.5708"/>
+      <origin xyz="0 0 0" rpy="0 0 -1.570796"/>
+      <geometry>
+        <mesh filename="package://xbot2_description/meshes/wheel.dae" />
+      </geometry>
+    </visual>
+    <inertial>
+      <origin xyz="0 0 0" rpy="0 0 -1.570796"/>
       <mass value="1.5"/>
       <inertia ixx=".001" ixy="0" ixz="0" iyy=".001" iyz="0" izz=".001" />
@@ -62,22 +92,22 @@
     <parent link="base_link"/>
     <child link="left_wheel"/>
-    <limit effort="5.2" velocity="21.05"/>
+    <limit effort="100000" velocity="1000"/>
     <joint_properties damping="0.0" friction="0.0"/>
   </joint>
   <link name="right_wheel">
     <collision name="collision">
-      <origin xyz="0 0 0" rpy="-1.5708  0 0"/>
-      <geometry>
-        <cylinder radius="0.095" length="0.04"/>
+      <origin xyz="0 0 0" rpy="-1.570796  0 0"/>
+      <geometry>
+        <cylinder radius="0.095" length="0.05"/>
       </geometry>
     </collision>
     <visual name="right_wheel_visual">
-      <origin xyz="0 0 0" rpy="0 0 1.5708"/>
-      <geometry>
-        <mesh filename="package://robot_sim_demo/meshes/wheel.dae" />
-      </geometry>
-    </visual>
-    <inertial>
-      <origin xyz="0 0 0" rpy="0 0 1.5708"/>
+      <origin xyz="0 0 0" rpy="0 0 1.570796"/>
+      <geometry>
+        <mesh filename="package://xbot2_description/meshes/wheel.dae" />
+      </geometry>
+    </visual>
+    <inertial>
+      <origin xyz="0 0 0" rpy="0 0 1.570796"/>
       <mass value="1.5"/>
       <inertia ixx=".001" ixy="0" ixz="0" iyy=".001" iyz="0" izz=".001" />
@@ -89,5 +119,5 @@
     <parent link="base_link"/>
     <child link="right_wheel"/>
-    <limit effort="5.2" velocity="21.05"/>
+    <limit effort="100000" velocity="1000"/>
     <joint_properties damping="0.0" friction="0.0"/>
   </joint>
@@ -99,14 +129,14 @@
     </inertial>
     <visual>
-      <origin xyz="0 0 0" rpy="0 0 1.5708" />
-      <geometry>
-        <mesh filename="package://robot_sim_demo/meshes/yaw_platform.stl" />
+      <origin xyz="0 0 0" rpy="0 0 1.570796" />
+      <geometry>
+        <mesh filename="package://xbot2_description/meshes/yaw_platform.stl" />
       </geometry>
       <material name="grey"/>
     </visual>
     <collision>
-      <origin xyz="0 0 0" rpy="0 0 1.5708" />
-      <geometry>
-        <mesh filename="package://robot_sim_demo/meshes/yaw_platform.stl" />
+      <origin xyz="0 0 0" rpy="0 0 1.570796" />
+      <geometry>
+        <box size="0.0 0.0 0.0"/>
       </geometry>
     </collision>
@@ -129,5 +159,5 @@
       <origin xyz="0 0 0" rpy="0 0 0" />
       <geometry>
-        <mesh filename="package://robot_sim_demo/meshes/pitch_platform.stl" />
+        <mesh filename="package://xbot2_description/meshes/pitch_platform.stl" />
       </geometry>
       <material name="grey"/>
@@ -136,5 +166,5 @@
       <origin xyz="0 0 0" rpy="0 0 0" />
       <geometry>
-        <mesh filename="package://robot_sim_demo/meshes/pitch_platform.stl" />
+        <box size="0.0 0.0 0.0"/>
       </geometry>
     </collision>
@@ -153,5 +183,5 @@
       <origin xyz="0 0 0" rpy="0 0 0"/>
       <geometry>
-        <mesh filename="package://robot_sim_demo/meshes/xtion_pro_camera.dae" />
+        <box size="0.0 0.0 0.0"/>
       </geometry>
     </collision>
@@ -159,5 +189,5 @@
       <origin xyz="0 0 0" rpy="0 0 0"/>
       <geometry>
-        <mesh filename="package://robot_sim_demo/meshes/xtion_pro_camera.dae" />
+        <mesh filename="package://xbot2_description/meshes/xtion_pro_camera.dae" />
       </geometry>
       <material name="gray"/>

Commit message: fix bugs that xbot2_description still remains

File: robot_sim_demo/urdf/robot.xacro (robot description, xacro)
@@ -5,10 +5,10 @@
   xmlns:xacro="http://ros.org/wiki/xacro"
   name="sick_tim">
-  <xacro:include filename="$(find xbot2_description)/urdf/sick_tim.urdf.xacro" />
+  <xacro:include filename="$(find robot_sim_demo)/urdf/sick_tim.urdf.xacro" />
   <xacro:sick_tim571 name="laser" ros_topic="scan"   />
-  <xacro:include filename="$(find xbot2_description)/urdf/materials.xacro" />
-  <xacro:include filename="$(find xbot2_description)/urdf/xbot2.urdf.xacro" />
-  <xacro:include filename="$(find xbot2_description)/urdf/xbot2.gazebo" />
+  <xacro:include filename="$(find robot_sim_demo)/urdf/materials.xacro" />
+  <xacro:include filename="$(find robot_sim_demo)/urdf/xbot2.urdf.xacro" />
+  <xacro:include filename="$(find robot_sim_demo)/urdf/xbot2.gazebo" />
   <xacro:xbot2_base/>
-  <!--xacro:include filename="$(find xbot2_description)/urdf/sick_tim.gazebo.xacro" /-->
+  <!--xacro:include filename="$(find robot_sim_demo)/urdf/sick_tim.gazebo.xacro" /-->
 </robot>

File: robot_sim_demo/urdf/sick_tim.urdf.xacro (robot description, xacro)
@@ -8,5 +8,5 @@
       length="0.06" width="0.06" height="0.079" mass="0.150" z_offset="0.05595"
       min_range="0.05" max_range="4.0"
-      mesh="package://xbot2_description/meshes/sick_tim310.stl" />
+      mesh="package://robot_sim_demo/meshes/sick_tim310.stl" />
   </xacro:macro>
   <xacro:macro name="sick_tim551" params="name ros_topic">
@@ -14,5 +14,5 @@
       length="0.06" width="0.06" height="0.086" mass="0.250" z_offset="0.06296"
       min_range="0.05" max_range="10.0"
-      mesh="package://xbot2_description/meshes/sick_tim551.stl" />
+      mesh="package://robot_sim_demo/meshes/sick_tim551.stl" />
   </xacro:macro>
   <xacro:macro name="sick_tim571" params="name ros_topic">
@@ -20,5 +20,5 @@
       length="0.06" width="0.06" height="0.086" mass="0.250" z_offset="0.02"
       min_range="0.05" max_range="25.0"
-      mesh="package://xbot2_description/meshes/sick_tim571.stl" />
+      mesh="package://robot_sim_demo/meshes/sick_tim571.stl" />
   </xacro:macro>
   <xacro:macro name="sick_tim" params="name ros_topic length width height mass z_offset min_range max_range mesh">

File: robot_sim_demo/urdf/xbot2.urdf.xacro (robot description, xacro)
@@ -21,5 +21,5 @@
       <origin xyz="0 0 0" rpy="0 0 0" />
       <geometry>
-        <mesh filename="package://xbot2_description/meshes/base_link.dae" />
+        <mesh filename="package://robot_sim_demo/meshes/base_link.dae" />
       </geometry>
     </visual>
@@ -78,5 +78,5 @@
       <origin xyz="0 0 0" rpy="0 0 -1.570796"/>
       <geometry>
-        <mesh filename="package://xbot2_description/meshes/wheel.dae" />
+        <mesh filename="package://robot_sim_demo/meshes/wheel.dae" />
       </geometry>
     </visual>
@@ -105,5 +105,5 @@
       <origin xyz="0 0 0" rpy="0 0 1.570796"/>
       <geometry>
-        <mesh filename="package://xbot2_description/meshes/wheel.dae" />
+        <mesh filename="package://robot_sim_demo/meshes/wheel.dae" />
       </geometry>
     </visual>
@@ -131,5 +131,5 @@
       <origin xyz="0 0 0" rpy="0 0 1.570796" />
       <geometry>
-        <mesh filename="package://xbot2_description/meshes/yaw_platform.stl" />
+        <mesh filename="package://robot_sim_demo/meshes/yaw_platform.stl" />
       </geometry>
       <material name="grey"/>
@@ -159,5 +159,5 @@
       <origin xyz="0 0 0" rpy="0 0 0" />
       <geometry>
-        <mesh filename="package://xbot2_description/meshes/pitch_platform.stl" />
+        <mesh filename="package://robot_sim_demo/meshes/pitch_platform.stl" />
       </geometry>
       <material name="grey"/>
@@ -189,5 +189,5 @@
       <origin xyz="0 0 0" rpy="0 0 0"/>
       <geometry>
-        <mesh filename="package://xbot2_description/meshes/xtion_pro_camera.dae" />
+        <mesh filename="package://robot_sim_demo/meshes/xtion_pro_camera.dae" />
       </geometry>
       <material name="gray"/>

Commit message: update xbot2-u model

File: robot_sim_demo/urdf/robot.xacro (robot description, xacro)
@@ -6,9 +6,10 @@
   name="sick_tim">
   <xacro:include filename="$(find robot_sim_demo)/urdf/sick_tim.urdf.xacro" />
-  <xacro:sick_tim571 name="laser" ros_topic="scan"   />
+  <!-- Choose your laser -->
+  <!--<xacro:sick_tim571 name="laser" ros_topic="scan"   />-->
+  <xacro:rplidarA2 name="laser" ros_topic="scan"   />
   <xacro:include filename="$(find robot_sim_demo)/urdf/materials.xacro" />
   <xacro:include filename="$(find robot_sim_demo)/urdf/xbot2.urdf.xacro" />
   <xacro:include filename="$(find robot_sim_demo)/urdf/xbot2.gazebo" />
   <xacro:xbot2_base/>
-  <!--xacro:include filename="$(find robot_sim_demo)/urdf/sick_tim.gazebo.xacro" /-->
 </robot>

File: robot_sim_demo/urdf/sick_tim.urdf.xacro (robot description, xacro)
@@ -4,4 +4,10 @@
   xmlns:sensor="http://playerstage.sourceforge.net/gazebo/xmlschema/#sensor"
   xmlns:xacro="http://ros.org/wiki/xacro">
+  <xacro:macro name="rplidarA2" params="name ros_topic">
+    <xacro:sick_tim name="${name}" ros_topic="${ros_topic}"
+      length="0.06" width="0.06" height="0.079" mass="0.150" z_offset="0.05595"
+      min_range="0.2" max_range="8.0"
+      mesh="package://robot_sim_demo/models/meshes/rplidar.dae" />
+  </xacro:macro>
   <xacro:macro name="sick_tim310" params="name ros_topic">
     <xacro:sick_tim name="${name}" ros_topic="${ros_topic}"

File: robot_sim_demo/urdf/xbot2.urdf.xacro (robot description, xacro)
@@ -14,7 +14,7 @@
   <link name="base_link">
     <inertial>
-      <origin  xyz="0.001 0 0.007" rpy="0 0 0" />
-      <mass value="30.0" />
-      <inertia ixx="1.734" ixy="0" ixz="0" iyy="1.734" iyz=".0" izz="1.0" />
+      <origin rpy="0 0 0" xyz="-0.015 0.0 0.0014" />
+      <mass value="35" />
+      <inertia ixx="0.6125" ixy="0.00495" ixz="0.0031" iyy="0.6426" iyz="-0.0017" izz="0.494" />
     </inertial>
     <visual>
@@ -66,5 +66,5 @@
     <parent link="base_link"/>
     <child link="laser_mount_link"/>
-    <origin rpy="0 3.1416 3.1416" xyz=".148 0 .253"/>
+    <origin rpy="0 0 0" xyz=".114 0 .17"/>
   </joint>
   <link name="imu_link"/>
@@ -77,5 +77,5 @@
   <link name="left_wheel">
     <collision name="collision">
-      <origin xyz="0 0 0" rpy="1.570796 0 0"/>
+      <origin xyz="0 0 0" rpy="1.57079632 0 0"/>
       <geometry>
         <cylinder radius="0.095" length="0.05"/>
@@ -83,5 +83,5 @@
     </collision>
     <visual name="left_wheel_visual">
-      <origin xyz="0 0 0" rpy="0 0 -1.570796"/>
+      <origin xyz="0 0 0" rpy="0 0 -1.57079632"/>
       <geometry>
         <mesh filename="package://robot_sim_demo/models/meshes/wheel.dae" />
@@ -89,20 +89,20 @@
     </visual>
     <inertial>
-      <origin xyz="0 0 0" rpy="0 0 -1.570796"/>
-      <mass value="1.5"/>
-      <inertia ixx=".001" ixy="0" ixz="0" iyy=".001" iyz="0" izz=".001" />
+      <origin rpy="0 0 0" xyz="0 0 0" />
+      <mass value="4.3542" />
+      <inertia ixx="0.0045" ixy="0" ixz="0" iyy="0.005" iyz="0" izz="0.0045" />
     </inertial>
   </link>
   <joint type="continuous" name="left_wheel_hinge">
     <axis xyz="0 1 0" rpy="0 0 0"/>
-    <origin xyz="0 0.245 .095" rpy="0 0 0"/>
+    <origin xyz="0 0.23 .095" rpy="0 0 0"/>
     <parent link="base_link"/>
     <child link="left_wheel"/>
-    <limit effort="5.2" velocity="2.0"/>
+    <limit effort="6" velocity="1.0"/>
     <joint_properties damping="0.0" friction="0.0"/>
   </joint>
   <link name="right_wheel">
     <collision name="collision">
-      <origin xyz="0 0 0" rpy="-1.570796  0 0"/>
+      <origin xyz="0 0 0" rpy="-1.57079632  0 0"/>
       <geometry>
         <cylinder radius="0.095" length="0.05"/>
@@ -110,5 +110,5 @@
     </collision>
     <visual name="right_wheel_visual">
-      <origin xyz="0 0 0" rpy="0 0 1.570796"/>
+      <origin xyz="0 0 0" rpy="0 0 1.57079632"/>
       <geometry>
         <mesh filename="package://robot_sim_demo/models/meshes/wheel.dae" />
@@ -116,32 +116,31 @@
     </visual>
     <inertial>
-      <origin xyz="0 0 0" rpy="0 0 1.570796"/>
-      <mass value="1.5"/>
-      <inertia ixx=".001" ixy="0" ixz="0" iyy=".001" iyz="0" izz=".001" />
+      <origin rpy="0 0 0" xyz="0 0 0" />
+      <mass value="4.3542" />
+      <inertia ixx="0.0045" ixy="0" ixz="0" iyy="0.005" iyz="0" izz="0.0045" />
     </inertial>
   </link>
   <joint type="continuous" name="right_wheel_hinge">
     <axis xyz="0 1 0" rpy="0 0 0"/>
-    <origin xyz="0 -0.245 .095" rpy="0 0 0"/>
+    <origin xyz="0 -0.23 .095" rpy="0 0 0"/>
     <parent link="base_link"/>
     <child link="right_wheel"/>
-    <limit effort="5.2" velocity="2.0"/>
+    <limit effort="6" velocity="1.0"/>
     <joint_properties damping="0.0" friction="0.0"/>
   </joint>
   <link name="yaw_platform">
     <inertial>
-      <origin  xyz="0 0 0" rpy="0 0 0" />
-      <mass value=".11" />
-      <inertia ixx="0.000826" ixy="0" ixz="0" iyy="0.0009211" iyz="0" izz="0.0002601" />
-    </inertial>
-    <visual>
-      <origin xyz="0 0 0" rpy="0 0 1.570796" />
-      <geometry>
-        <mesh filename="package://robot_sim_demo/models/meshes/yaw_platform.stl" />
-      </geometry>
-      <material name="grey"/>
+      <mass value="1e-5" />
+      <origin xyz="0 0 0" rpy="0 0 0"/>
+      <inertia ixx="1e-6" ixy="0" ixz="0" iyy="1e-6" iyz="0" izz="1e-6" />
+    </inertial>
+    <visual>
+      <origin xyz="0 0 0" rpy="0 0 1.57079632" />
+      <geometry>
+        <mesh filename="package://robot_sim_demo/models/meshes/yaw_platform.dae" />
+      </geometry>
     </visual>
     <collision>
-      <origin xyz="0 0 0" rpy="0 0 1.570796" />
+      <origin xyz="0 0 0" rpy="0 0 1.57079632" />
       <geometry>
         <box size="0.1 0.1 0.1"/>
@@ -153,20 +152,19 @@
     <parent link="base_link"/>
     <child link="yaw_platform"/>
-    <origin rpy="0 0 0" xyz="0 0 1.07"/>
+    <origin rpy="0 0 0" xyz="0 0 1.305"/>
     <limit effort="100" velocity="100" lower="-1.57" upper="1.57" />
-    <dynamics damping="0.0" friction="5.0"/>
+    <dynamics damping="0.0" friction="10.0"/>
   </joint>
   <link name="pitch_platform">
     <inertial>
-      <origin  xyz="0 0 0" rpy="0 0 0" />
-      <mass value=".05" />
-      <inertia ixx="0.0001" ixy="0" ixz="0" iyy="0.00001" iyz="0" izz="0.0001" />
+      <mass value="1e-5" />
+      <origin xyz="0 0 0" rpy="0 0 0"/>
+      <inertia ixx="1e-6" ixy="0" ixz="0" iyy="1e-6" iyz="0" izz="1e-6" />
     </inertial>
     <visual>
       <origin xyz="0 0 0" rpy="0 0 0" />
       <geometry>
-        <mesh filename="package://robot_sim_demo/models/meshes/pitch_platform.stl" />
-      </geometry>
-      <material name="grey"/>
+        <mesh filename="package://robot_sim_demo/models/meshes/pitch_platform.dae" />
+      </geometry>
     </visual>
     <collision>
@@ -181,7 +179,7 @@
     <parent link="yaw_platform"/>
     <child link="pitch_platform"/>
-    <origin rpy="0 0 0" xyz="0 0 .02"/>
+    <origin rpy="0 0 0" xyz="0 0 0"/>
     <limit effort="100" velocity="100" lower="-1.57" upper="1.57" />
-    <dynamics damping="0.0" friction="5.0"/>
+    <dynamics damping="0.0" friction="10.0"/>
   </joint>
   <!-- Camera -->
@@ -196,7 +194,7 @@
       <origin xyz="0 0 0" rpy="0 0 0"/>
       <geometry>
-        <mesh filename="package://robot_sim_demo/models/meshes/xtion_pro_camera.dae" />
-      </geometry>
-      <material name="gray"/>
+        <!--<mesh filename="package://robot_sim_demo/models/meshes/xtion_pro_camera.dae" />-->
+        <mesh filename="package://robot_sim_demo/models/meshes/realsense.dae" />
+      </geometry>
     </visual>
     <inertial>
@@ -208,5 +206,5 @@
   <joint name="camera_joint" type="fixed">
     <axis xyz="0 1 0" />
-    <origin xyz="0 0 .08" rpy="0 0 0"/>
+    <origin xyz="-0.005 0 .06" rpy="0 0 0"/>
     <parent link="pitch_platform"/>
     <child link="camera_link"/>
