Commit message: 添加urdf_demo

File: urdf_demo/urdf/mycar_color_geometry.urdf (robot description, URDF)
Before this commit: robot mycar, 4 links, 3 joints
Links:
- link rplidar: geometry collision cylinder length=.04 radius=0.035; visual mesh filename=package://urdf_demo/urdf/rplidar.dae

Commit message: 更新urdf_demo

File: urdf_demo/urdf/mycar_color_geometry.urdf (robot description, URDF)
Before this commit: robot mycar, 4 links, 3 joints
Joints:
- joint left: origin xyz=0 0.2 0.07 rpy=-1.57075 0 0 -> xyz=0 0.2 0.07 rpy=0 0 0
- joint right: origin xyz=0 -0.2 0.07 rpy=1.57075  0  0 -> xyz=0 -0.2 0.07 rpy=0  0  0

File: urdf_demo/urdf/mycar_link_position.urdf (robot description, URDF)
Before this commit: robot mycar, 4 links, 3 joints
Joints:
- joint left: origin xyz=0 0.2 0.07 rpy=-1.57075 0 0 -> xyz=0 0.2 0.07 rpy=0 0 0
- joint right: origin xyz=0 -0.2 0.07 rpy=1.57075  0  0 -> xyz=0 -0.2 0.07 rpy=0  0  0
